File: starclip/starclip.kicad_sch (KiCad schematic)
At the start: 2 parts, among them J7 Sparkle Motion Mini, SW1 SW_SPST

Commit message: project schematic
Parts:
- added BT1: Battery_Cell, symbol Device:Battery_Cell
- added D13: WS2812B, LED_SMD:LED_WS2812B_PLCC4_5.0x5.0mm_P3.2mm, symbol LED:WS2812B
- added J8: MiniBoost 5V, symbol Connector_Generic:Conn_01x04
Connections:
- net starLeft/5V: now also J7.4 (Pin_4), D13.1 (VDD), J8.3 (Pin_3)
- net starLeft/DATA: now also J7.2 (Pin_2)
- net starLeft/GND: now also J7.1 (Pin_1), SW1.1 (A), BT1.2 (-), D13.3 (VSS), J8.2 (Pin_2)
- net at J7.3 (Pin_3): now also D13.4 (DIN)
- net at SW1.2 (B): now also J8.4 (Pin_4)
- new net: BT1.1 (+), J8.1 (Pin_1)
- new net starRight/DATA: D13.2 (DOUT)
Other:
- sheet star renamed starLeft
- added sheet starRight (star.kicad_sch)
- note added: "visual representation of the led chain within the bow ->"
- moved on the sheet: SW1
